Commit message: a couple changes to get TF2 working so I could use SLAM.

File: kobuki_description/urdf/kobuki.urdf.xacro (robot description, xacro)
@@ -22,7 +22,7 @@
       -->
     <joint name="base_joint" type="fixed">
-      <origin xyz="0 0 0.0102" rpy="0 0 0" />
-      <parent link="base_footprint"/>
-      <child link="base_link" />
+      <origin xyz="0 0 -0.0102" rpy="0 0 0" />
+      <parent link="base_link"/>
+      <child link="base_footprint" />
     </joint>
     <link name="base_link">

File: kobuki_description/urdf/kobuki_gazebo.urdf.xacro (robot description, xacro)
@@ -182,5 +182,5 @@
         <!-- output -->
         <publish_odom>true</publish_odom>
-        <publish_odom_tf>false</publish_odom_tf>
+        <publish_odom_tf>true</publish_odom_tf>
         <publish_wheel_tf>false</publish_wheel_tf>
         <odometry_topic>odom</odometry_topic>
